File: universerial.kicad_pcb (KiCad board)
At the start: 2 copper layers, 19 parts, among them J1 USB_A, J2 Conn_01x06, U1 CH340G, Y1 12MHz

Commit message: Organize PCB.
Parts:
- moved R2 39.6 mm to (174.9, 86.4), turned to 270 degrees
- moved R3 39.1 mm to (180.3, 86.4), turned to 270 degrees
- moved J2 38.5 mm to (201.9, 96.5)
- moved D4 36.4 mm to (182.9, 94.5), turned to 180 degrees
- moved C6 33.5 mm to (168.9, 86.4)
- moved Y1 30.7 mm to (142.2, 95.2)
- moved D3 28.9 mm to (171.4, 94.0)
- moved J1 28.7 mm to (116.3, 97.5)
- moved U1 27.2 mm to (160.0, 91.4)
- moved D5 25.9 mm to (167.3, 96.5)
- moved C5 23.1 mm to (148.6, 86.4)
- moved C2 22.9 mm to (138.4, 86.4)
- moved R4 19.3 mm to (186.7, 102.9)
- moved R1 18.4 mm to (158.4, 109.2)
- moved C1 18.2 mm to (133.3, 86.4)
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Routing:
- net GND: track 0.00 -> 6.47 mm
Other:
- board outline added: 114.3 x 38.1 mm
- board text added: "Biel A. P."
- board text added: "Universerial"

Commit message: Finish PCB.
Routing:
- net GND: track 6.47 -> 188.9 mm
- net +5V: track 0.00 -> 119.5 mm
- net Net-(C6-Pad1): track 0.00 -> 101.9 mm
- net Net-(D4-Pad1): track 0.00 -> 70.5 mm
- net Net-(J1-Pad3): track 0.00 -> 56.6 mm
- net Net-(J1-Pad2): track 0.00 -> 52.0 mm
- net +3V3: track 0.00 -> 51.9 mm, vias 0 -> 2
- net Net-(D2-Pad1): track 0.00 -> 38.8 mm
- net Net-(C3-Pad1): track 0.00 -> 20.6 mm
- net Net-(C4-Pad1): track 0.00 -> 13.4 mm
- net Net-(J2-Pad4): track 0.00 -> 12.3 mm
- net Net-(D4-Pad2): track 0.00 -> 8.54 mm
- net Net-(D2-Pad2): track 0.00 -> 7.11 mm
- net Net-(D1-Pad1): track 0.00 -> 5.50 mm
- net Net-(D3-Pad1): track 0.00 -> 4.57 mm
